File: pcbs/brolga.kicad_pcb (KiCad board)
At the start: 2 copper layers, 127.9 x 81.7 mm, 23 parts, among them J1 Jumper, J2 Jumper, J3 Jumper

Commit message: fixes
Routing:
- net GND: track 689.9 -> 0.00 mm
- net SW7: track 75.8 -> 85.8 mm
- net SW6: track 125.1 -> 135.1 mm
- added copper zone on B.Cu, net GND
- added copper zone on F.Cu, net GND
Other:
- board text added: "'tis death i wed"
- board text added: "room for art in future iteration"
