File: brolga/beryllish.kicad_pcb (KiCad board)
At the start: 2 copper layers, 127.9 x 81.7 mm, 23 parts, among them J1 Jumper, J2 Jumper, J3 Jumper

Commit message: minor refactor
Connections:
- MCU1 pad : (no net) -> GND
Routing:
- net GND: track 0.00 -> 53.6 mm
Changed lines of the file:
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@@
       ))
     (pad "" smd custom locked (at -11.43 -5.842) (size 0.1 0.1) (layers "F.Cu" "F.Mask")
-      (clearance 0.1) (zone_connect 0)
+      (net 1 "GND") (clearance 0.1) (zone_connect 0)
       (options (clearance outline) (anchor rect))
       (primitives
@@
       ))
     (pad "" smd custom locked (at -8.89 6.35 180) (size 0.25 1) (layers "F.Cu")
-      (zone_connect 0)
+      (net 1 "GND") (zone_connect 0)
       (options (clearance outline) (anchor rect))
       (primitives
@@
       ))
     (pad "" smd custom locked (at -6.35 5.842 180) (size 0.1 0.1) (layers "F.Cu" "F.Mask")
-      (clearance 0.1) (zone_connect 0)
+      (net 1 "GND") (clearance 0.1) (zone_connect 0)
       (options (clearance outline) (anchor rect))
       (primitives
@@
       ))
     (pad "" smd custom locked (at -8.89 5.842 180) (size 0.1 0.1) (layers "F.Cu" "F.Mask")
-      (clearance 0.1) (zone_connect 0)
+      (net 1 "GND") (clearance 0.1) (zone_connect 0)
       (options (clearance outline) (anchor rect))
       (primitives
@@
       (net 1 "GND"))
     (pad "2" smd custom locked (at -11.43 -4.826) (size 1.2 0.5) (layers "F.Cu" "F.Mask")
-      (clearance 0.1) (zone_connect 0)
+      (net 1 "GND") (clearance 0.1) (zone_connect 0)
       (options (clearance outline) (anchor rect))
       (primitives
@@
       ))
     (pad "2" smd custom locked (at -11.43 4.826 180) (size 1.2 0.5) (layers "B.Cu" "B.Mask")
-      (clearance 0.1) (zone_connect 0)
+      (net 1 "GND") (clearance 0.1) (zone_connect 0)
       (options (clearance outline) (anchor rect))
       (primitives
@@
       ))
     (pad "21" smd custom locked (at -6.35 -4.826) (size 1.2 0.5) (layers "B.Cu" "B.Mask")
-      (clearance 0.1) (zone_connect 0)
+      (net 1 "GND") (clearance 0.1) (zone_connect 0)
       (options (clearance outline) (anchor rect))
       (primitives
@@
       ))
     (pad "21" smd custom locked (at -6.35 4.826 180) (size 1.2 0.5) (layers "F.Cu" "F.Mask")
-      (clearance 0.1) (zone_connect 0)
+      (net 1 "GND") (clearance 0.1) (zone_connect 0)
       (options (clearance outline) (anchor rect))
       (primitives
@@
       ))
     (pad "21" smd custom locked (at -6.35 0.762 180) (size 0.25 0.25) (layers "F.Cu")
-      (zone_connect 0)
+      (net 1 "GND") (zone_connect 0)
       (options (clearance outline) (anchor circle))
       (primitives
@@
       (net 1 "GND"))
     (pad "22" smd custom locked (at -8.89 0.762 180) (size 0.25 0.25) (layers "F.Cu")
-      (zone_connect 0)
+      (net 1 "GND") (zone_connect 0)
       (options (clearance outline) (anchor circle))
       (primitives
@@
       (net 1 "GND"))
     (pad "22" smd custom locked (at -8.89 4.826 180) (size 1.2 0.5) (layers "F.Cu" "F.Mask")
-      (clearance 0.1) (zone_connect 0)
+      (net 1 "GND") (clearance 0.1) (zone_connect 0)
       (options (clearance outline) (anchor rect))
       (primitives
@@
       ))
     (pad "22" smd custom locked (at -8.89 -4.826) (size 1.2 0.5) (layers "B.Cu" "B.Mask")
-      (clearance 0.1) (zone_connect 0)
+      (net 1 "GND") (clearance 0.1) (zone_connect 0)
       (options (clearance outline) (anchor rect))
       (primitives
@@
       ))
     (pad "22" smd custom locked (at -8.89 0.762 180) (size 0.25 0.25) (layers "B.Cu")
-      (zone_connect 0)
+      (net 1 "GND") (zone_connect 0)
       (options (clearance outline) (anchor circle))
       (primitives
@@
     (effects (font (size 1 1) (thickness 0.15)))
   )
+  (segment (start 56.11638 104.91962) (end 55.372 105.664) (width 0.25) (layer "F.Cu") (net 1))
+  (segment (start 55.372 105.664) (end 55.372 106.68) (width 0.25) (layer "F.Cu") (net 1))
+  (segment (start 55.372 106.68) (end 57.404 108.712) (width 0.25) (layer "F.Cu") (net 1))
+  (segment (start 57.404 108.712) (end 61.976 108.712) (width 0.25) (layer "F.Cu") (net 1))
+  (segment (start 61.976 108.712) (end 61.976 116.105) (width 0.25) (layer "F.Cu") (net 1))
+  (segment (start 57.018514 104.91962) (end 56.11638 104.91962) (width 0.25) (layer "F.Cu") (net 1))
+  (segment (start 61.976 116.105) (end 63.219 117.348) (width 0.25) (layer "F.Cu") (net 1))
+  (segment (start 92.518134 109.67) (end 92.213623 109.365489) (width 0.25) (layer "B.Cu") (net 1))
+  (segment (start 69.596 119.126) (end 69.342 119.38) (width 0.25) (layer "B.Cu") (net 1))
+  (segment (start 69.342 119.38) (end 68.807 119.38) (width 0.25) (layer "B.Cu") (net 1))
+  (segment (start 70.212511 109.365489) (end 69.596 109.982) (width 0.25) (layer "B.Cu") (net 1))
+  (segment (start 69.596 109.982) (end 69.596 119.126) (width 0.25) (layer "B.Cu") (net 1))
+  (segment (start 92.213623 109.365489) (end 70.212511 109.365489) (width 0.25) (layer "B.Cu") (net 1))
+  (segment (start 68.807 119.38) (end 68.299 118.872) (width 0.25) (layer "B.Cu") (net 1))
   (segment (start 64.516 116.105) (end 65.759 117.348) (width 0.25) (layer "F.Cu") (net 2))
   (segment (start 64.516 109.728) (end 64.516 116.105) (width 0.25) (layer "F.Cu") (net 2))
@@
   (segment (start 166.58578 49.528113) (end 57.792889 49.528113) (width 0.25) (layer "B.Cu") (net 4))
   (segment (start 55.758624 127.215036) (end 55.758528 127.215132) (width 0.25) (layer "B.Cu") (net 4))
-  (segment (start 166.624 49.489893) (end 166.58578 49.528113) (width 0.25) (layer "B.Cu") (net 4))
   (segment (start 55.758528 127.215132) (end 57.575396 129.032) (width 0.25) (layer "B.Cu") (net 4))
-  (segment (start 166.624 49.624) (end 166.624 49.489893) (width 0.25) (layer "B.Cu") (net 4))
   (segment (start 57.792889 49.528113) (end 55.75483 51.566172) (width 0.25) (layer "B.Cu") (net 4))
   (segment (start 55.758624 51.569766) (end 55.758624 127.215036) (width 0.25) (layer "B.Cu") (net 4))
@@
     (polygon
       (pts
-        (xy 184.658 46.736)
-        (xy 185.42 132.842)
-        (xy 48.006 132.334)
-        (xy 47.498 45.466)
+        (xy 185.674 44.196)
+        (xy 186.69 132.588)
+        (xy 50.038 133.35)
+        (xy 50.8 43.434)
       )
     )

Commit message: more fixes
Parts:
- added B+: MountingHole_Pad, kbd:1pin_conn, F.Cu at (57.7, 110.5)
- added B-: MountingHole_Pad, kbd:1pin_conn, F.Cu at (57.7, 125.7)
Connections:
- MCU1 pad : GND -> (no net)
Routing:
- net GND: track 53.6 -> 50.5 mm
Changed lines of the file:
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@@
   (net 21 "SW16")
   (net 22 "SW17")
+  (footprint "kbd:1pin_conn" (layer "F.Cu")
+    (at 57.658 125.73 90)
+    (descr "Resitance 3 pas")
+    (tags "R")
+    (autoplace_cost180 10)
+    (attr through_hole)
+    (fp_text reference "B-" (at 1.778 0 90) (layer "F.SilkS")
+      (effects (font (size 0.6 0.6) (thickness 0.15)))
+    )
+    (fp_text value "MountingHole_Pad" (at 0 -1.4605 90) (layer "F.Fab") hide
+      (effects (font (size 0.5 0.5) (thickness 0.125)))
+    )
+    (fp_line (start -1 1) (end -1 -1) (layer "B.SilkS") (width 0.15))
+    (fp_line (start 1 1) (end -1 1) (layer "B.SilkS") (width 0.15))
+    (fp_line (start -1 -1) (end 1 -1) (layer "B.SilkS") (width 0.15))
+    (fp_line (start 1 -1) (end 1 1) (layer "B.SilkS") (width 0.15))
+    (fp_line (start 1 -1) (end -1 -1) (layer "F.SilkS") (width 0.15))
+    (fp_line (start -1 1) (end 1 1) (layer "F.SilkS") (width 0.15))
+    (fp_line (start -1 -1) (end -1 1) (layer "F.SilkS") (width 0.15))
+    (fp_line (start 1 1) (end 1 -1) (layer "F.SilkS") (width 0.15))
+    (pad "1" thru_hole circle locked (at 0 0 90) (size 1.397 1.397) (drill 0.8128) (layers *.Cu *.Mask "F.SilkS")
+      (net 1 "GND"))
+    (model "discret/resistor.wrl"
+      (offset (xyz 0 0 0))
+      (scale (xyz 0.3 0.3 0.3))
+      (rotate (xyz 0 0 0))
+    )
+    (model "Resistors_ThroughHole.3dshapes/Resistor_Horizontal_RM10mm.wrl"
+      (offset (xyz 0 0 0))
+      (scale (xyz 0.2 0.2 0.2))
+      (rotate (xyz 0 0 0))
+    )
+  )
   (footprint "lib:Jumper" (layer "F.Cu")
     (at 57.018514 105.42 -90)
@@
       (net 12 "VCC"))
   )
+  (footprint "kbd:1pin_conn" (layer "F.Cu")
+    (at 57.658 110.49 90)
+    (descr "Resitance 3 pas")
+    (tags "R")
+    (autoplace_cost180 10)
+    (attr through_hole)
+    (fp_text reference "B+" (at -1.778 0 90) (layer "F.SilkS")
+      (effects (font (size 0.6 0.6) (thickness 0.15)))
+    )
+    (fp_text value "MountingHole_Pad" (at 0 -1.4605 90) (layer "F.Fab") hide
+      (effects (font (size 0.5 0.5) (thickness 0.125)))
+    )
+    (fp_line (start -1 1) (end -1 -1) (layer "B.SilkS") (width 0.15))
+    (fp_line (start 1 -1) (end 1 1) (layer "B.SilkS") (width 0.15))
+    (fp_line (start 1 1) (end -1 1) (layer "B.SilkS") (width 0.15))
+    (fp_line (start -1 -1) (end 1 -1) (layer "B.SilkS") (width 0.15))
+    (fp_line (start 1 1) (end 1 -1) (layer "F.SilkS") (width 0.15))
+    (fp_line (start -1 -1) (end -1 1) (layer "F.SilkS") (width 0.15))
+    (fp_line (start -1 1) (end 1 1) (layer "F.SilkS") (width 0.15))
+    (fp_line (start 1 -1) (end -1 -1) (layer "F.SilkS") (width 0.15))
+    (pad "1" thru_hole circle locked (at 0 0 90) (size 1.397 1.397) (drill 0.8128) (layers *.Cu *.Mask "F.SilkS"))
+    (model "discret/resistor.wrl"
+      (offset (xyz 0 0 0))
+      (scale (xyz 0.3 0.3 0.3))
+      (rotate (xyz 0 0 0))
+    )
+    (model "Resistors_ThroughHole.3dshapes/Resistor_Horizontal_RM10mm.wrl"
+      (offset (xyz 0 0 0))
+      (scale (xyz 0.2 0.2 0.2))
+      (rotate (xyz 0 0 0))
+    )
+  )
   (footprint "pretty:SW_MX_choc" (layer "F.Cu")
     (at 141.243999 60.32)
@@
       ))
     (pad "" smd custom locked (at -11.43 -5.842) (size 0.1 0.1) (layers "F.Cu" "F.Mask")
-      (net 1 "GND") (clearance 0.1) (zone_connect 0)
+      (clearance 0.1) (zone_connect 0)
       (options (clearance outline) (anchor rect))
       (primitives
@@
       ))
     (pad "" smd custom locked (at -8.89 6.35 180) (size 0.25 1) (layers "F.Cu")
-      (net 1 "GND") (zone_connect 0)
+      (zone_connect 0)
       (options (clearance outline) (anchor rect))
       (primitives
@@
       ))
     (pad "" smd custom locked (at -6.35 5.842 180) (size 0.1 0.1) (layers "F.Cu" "F.Mask")
-      (net 1 "GND") (clearance 0.1) (zone_connect 0)
+      (clearance 0.1) (zone_connect 0)
       (options (clearance outline) (anchor rect))
       (primitives
@@
       ))
     (pad "" smd custom locked (at -8.89 5.842 180) (size 0.1 0.1) (layers "F.Cu" "F.Mask")
-      (net 1 "GND") (clearance 0.1) (zone_connect 0)
+      (clearance 0.1) (zone_connect 0)
       (options (clearance outline) (anchor rect))
       (primitives
@@
     (effects (font (size 1 1) (thickness 0.15)))
   )
-  (segment (start 56.11638 104.91962) (end 55.372 105.664) (width 0.25) (layer "F.Cu") (net 1))
-  (segment (start 55.372 105.664) (end 55.372 106.68) (width 0.25) (layer "F.Cu") (net 1))
-  (segment (start 55.372 106.68) (end 57.404 108.712) (width 0.25) (layer "F.Cu") (net 1))
-  (segment (start 57.404 108.712) (end 61.976 108.712) (width 0.25) (layer "F.Cu") (net 1))
-  (segment (start 61.976 108.712) (end 61.976 116.105) (width 0.25) (layer "F.Cu") (net 1))
-  (segment (start 57.018514 104.91962) (end 56.11638 104.91962) (width 0.25) (layer "F.Cu") (net 1))
-  (segment (start 61.976 116.105) (end 63.219 117.348) (width 0.25) (layer "F.Cu") (net 1))
+  (segment (start 58.166 127.254) (end 57.658 126.746) (width 0.25) (layer "B.Cu") (net 1))
   (segment (start 92.518134 109.67) (end 92.213623 109.365489) (width 0.25) (layer "B.Cu") (net 1))
   (segment (start 69.596 119.126) (end 69.342 119.38) (width 0.25) (layer "B.Cu") (net 1))
+  (segment (start 61.722 127.254) (end 58.166 127.254) (width 0.25) (layer "B.Cu") (net 1))
   (segment (start 69.342 119.38) (end 68.807 119.38) (width 0.25) (layer "B.Cu") (net 1))
+  (segment (start 61.976 127) (end 61.722 127.254) (width 0.25) (layer "B.Cu") (net 1))
+  (segment (start 61.976 117.602) (end 61.976 127) (width 0.25) (layer "B.Cu") (net 1))
+  (segment (start 57.658 126.746) (end 57.658 125.73) (width 0.25) (layer "B.Cu") (net 1))
   (segment (start 70.212511 109.365489) (end 69.596 109.982) (width 0.25) (layer "B.Cu") (net 1))
+  (segment (start 63.219 117.348) (end 62.23 117.348) (width 0.25) (layer "B.Cu") (net 1))
   (segment (start 69.596 109.982) (end 69.596 119.126) (width 0.25) (layer "B.Cu") (net 1))
   (segment (start 92.213623 109.365489) (end 70.212511 109.365489) (width 0.25) (layer "B.Cu") (net 1))
+  (segment (start 62.23 117.348) (end 61.976 117.602) (width 0.25) (layer "B.Cu") (net 1))
   (segment (start 68.807 119.38) (end 68.299 118.872) (width 0.25) (layer "B.Cu") (net 1))
   (segment (start 64.516 116.105) (end 65.759 117.348) (width 0.25) (layer "F.Cu") (net 2))
@@
   (segment (start 57.018514 105.92038) (end 60.70838 105.92038) (width 0.25) (layer "F.Cu") (net 2))
   (segment (start 60.70838 105.92038) (end 64.516 109.728) (width 0.25) (layer "F.Cu") (net 2))
-  (segment (start 58.674 115.343) (end 58.674 108.458) (width 0.25) (layer "B.Cu") (net 3))
   (segment (start 93.472 108.712) (end 93.472 109.728) (width 0.25) (layer "B.Cu") (net 3))
   (segment (start 93.472 109.716894) (end 93.518894 109.67) (width 0.25) (layer "B.Cu") (net 3))
   (segment (start 60.679 117.348) (end 58.674 115.343) (width 0.25) (layer "B.Cu") (net 3))
+  (segment (start 58.681011 115.335989) (end 58.681011 108.465011) (width 0.25) (layer "B.Cu") (net 3))
   (segment (start 93.472 120.65762) (end 93.472 109.716894) (width 0.25) (layer "B.Cu") (net 3))
   (segment (start 58.928 108.204) (end 92.964 108.204) (width 0.25) (layer "B.Cu") (net 3))
   (segment (start 92.964 108.204) (end 93.472 108.712) (width 0.25) (layer "B.Cu") (net 3))
   (segment (start 58.674 108.458) (end 58.928 108.204) (width 0.25) (layer "B.Cu") (net 3))
+  (segment (start 58.681011 108.465011) (end 58.674 108.458) (width 0.25) (layer "B.Cu") (net 3))
+  (segment (start 58.674 115.343) (end 58.681011 115.335989) (width 0.25) (layer "B.Cu") (net 3))
   (segment (start 93.472 120.65762) (end 93.585184 120.65762) (width 0.25) (layer "B.Cu") (net 3))
   (segment (start 174.724 57.424) (end 179.324 57.424) (width 0.25) (layer "F.Cu") (net 4))
